Commit message: 加入碰撞属性

File: src/fishbot_description/urdf/fishbot/actuator/caster.urdf.xacro (robot description, xacro)
@@ -12,4 +12,13 @@
                 </material>
             </visual>
+            <collision>
+                <origin xyz="0.0 0.0 0.0" rpy="0.0 0.0 0.0" />
+                <geometry>
+                    <sphere radius="0.016" />
+                </geometry>
+                <material name="yellow">
+                    <color rgba="1.0 1.0 0.0 0.8" />
+                </material>
+            </collision>
         </link>
         <joint name="${caster_name}_joint" type="fixed">

File: src/fishbot_description/urdf/fishbot/actuator/wheel.urdf.xacro (robot description, xacro)
@@ -12,4 +12,13 @@
                 </material>
             </visual>
+            <collision>
+                <origin xyz="0.0 0.0 0.0" rpy="1.57079 0.0 0.0" />
+                <geometry>
+                    <cylinder radius="0.032" length="0.04" />
+                </geometry>
+                <material name="yellow">
+                    <color rgba="1.0 1.0 0.0 0.8" />
+                </material>
+            </collision>
         </link>
         <joint name="${wheel_name}_joint" type="continuous">

File: src/fishbot_description/urdf/fishbot/base.urdf.xacro (robot description, xacro)
@@ -2,4 +2,5 @@
 <robot xmlns:xacro="http://www.ros.org/wiki/xacro">
     <xacro:macro name="base_xacro" params="length radius">
+        <link name="base_footprint" />
         <link name="base_link">
             <visual>
@@ -12,5 +13,19 @@
                 </material>
             </visual>
+            <collision>
+                <origin xyz="0.0 0.0 0.0" rpy="0.0 0.0 0.0" />
+                <geometry>
+                    <cylinder radius="${radius}" length="${length}" />
+                </geometry>
+                <material name="white">
+                    <color rgba="1.0 1.0 1.0 0.5" />
+                </material>
+            </collision>
         </link>
+        <joint name="joint_name" type="fixed">
+            <origin xyz="0.0 0.0 ${length/2.0+0.032-0.01}" rpy="0.0 0.0 0.0" />
+            <parent link="base_footprint" />
+            <child link="base_link" />
+        </joint>
     </xacro:macro>
 </robot>

File: src/fishbot_description/urdf/fishbot/sensor/camera.urdf.xacro (robot description, xacro)
@@ -12,4 +12,13 @@
                 </material>
             </visual>
+            <collision>
+                <origin xyz="0.0 0.0 0.0" rpy="0.0 0.0 0.0" />
+                <geometry>
+                    <box size="0.02 0.02 0.02" />
+                </geometry>
+                <material name="black">
+                    <color rgba="0.0 0.0 0.0 0.8" />
+                </material>
+            </collision>
         </link>
         <joint name="camera_joint" type="fixed">

File: src/fishbot_description/urdf/fishbot/sensor/imu.urdf.xacro (robot description, xacro)
@@ -12,4 +12,13 @@
                 </material>
             </visual>
+            <collision>
+                <origin xyz="0.0 0.0 0.0" rpy="0.0 0.0 0.0" />
+                <geometry>
+                    <box size="0.02 0.02 0.02" />
+                </geometry>
+                <material name="black">
+                    <color rgba="0.0 0.0 0.0 0.8" />
+                </material>
+            </collision>
         </link>
         <joint name="imu_joint" type="fixed">

File: src/fishbot_description/urdf/fishbot/sensor/laser.urdf.xacro (robot description, xacro)
@@ -6,5 +6,5 @@
                 <origin xyz="0.0 0.0 0.0" rpy="0.0 0.0 0.0" />
                 <geometry>
-                    <cylinder radius="0.01" length="0.10"/>
+                    <cylinder radius="0.01" length="0.10" />
                 </geometry>
                 <material name="black">
@@ -23,4 +23,13 @@
                 </material>
             </visual>
+            <collision>
+                <origin xyz="0.0 0.0 0.0" rpy="0.0 0.0 0.0" />
+                <geometry>
+                    <cylinder radius="0.02" length="0.02" />
+                </geometry>
+                <material name="black">
+                    <color rgba="0.0 0.0 0.0 1.0" />
+                </material>
+            </collision>
         </link>
         <joint name="laser_joint" type="fixed">

Commit message: 加入gazebo标签

File: src/fishbot_description/urdf/fishbot/actuator/caster.urdf.xacro (robot description, xacro)
@@ -31,4 +31,10 @@
             <axis xyz="0.0 1.0 0.0" />
         </joint>
+        <gazebo reference="${caster_name}_link">
+            <mu1 value="0.0" />
+            <mu2 value="0.0" />
+            <kp value="100000000.0" />
+            <kd value="1.0" />
+        </gazebo>
     </xacro:macro>
 </robot>

File: src/fishbot_description/urdf/fishbot/actuator/wheel.urdf.xacro (robot description, xacro)
@@ -31,4 +31,10 @@
             <axis xyz="0.0 1.0 0.0" />
         </joint>
+        <gazebo reference="${wheel_name}_link">
+            <mu1 value="20.0" />
+            <mu2 value="20.0" />
+            <kp value="100000000.0" />
+            <kd value="1.0" />
+        </gazebo>
     </xacro:macro>
 </robot>

File: src/fishbot_description/urdf/fishbot/sensor/laser.urdf.xacro (robot description, xacro)
@@ -47,4 +47,10 @@
             <origin xyz="${xyz}" rpy="0.0 0.0 0.0" />
         </joint>
+        <gazebo reference='laser_cylinder_link'>
+            <material>Gazebo/Black</material>
+        </gazebo>
+        <gazebo reference='laser_link'>
+            <material>Gazebo/Black</material>
+        </gazebo>
     </xacro:macro>
 </robot>
