Commit message: 加入深度相机

File: src/fishbot_description/urdf/fishbot/sensor/camera.urdf.xacro (robot description, xacro)
@@ -25,4 +25,6 @@
             <xacro:box_inertia m="0.10" w="0.02" h="0.10" d="0.02" />
         </link>
+        <link name="camera_optical_link">
+        </link>
         <joint name="camera_joint" type="fixed">
             <parent link="base_link" />
@@ -30,4 +32,9 @@
             <origin xyz="${xyz}" rpy="0.0 0.0 0.0" />
         </joint>
+        <joint name="camera_optical_joint" type="fixed">
+            <parent link="camera_link" />
+            <child link="camera_optical_link" />
+            <origin xyz="0 0 0" rpy="${-pi/2} 0.0 ${-pi/2}" />
+        </joint>
     </xacro:macro>
 </robot>
